Commit message: [DCL-46] Moved the stick collision data inside of the chasis link

File: entity_files/drone_stick.urdf (robot description, URDF)
Before this commit: robot drone_simple, 6 links, 5 joints
Links:
- removed link stick
- link chasis: geometry collision cylinder length=0.15 radius=0.4; collision cylinder length=1.2 radius=0.02
Joints:
- removed joint stick_to_chasis
