Commit message: [DCL-39] Fix building collision tags

File: entity_files/building_long.urdf (robot description, URDF)
Before this commit: robot building_long, 1 links, 0 joints
Links:
- link building: geometry collision box size=1 5 2; visual box size=1 5 2

File: entity_files/building_short.urdf (robot description, URDF)
Before this commit: robot building_short, 1 links, 0 joints
Links:
- link building: geometry collision box size=2 2 2; visual box size=2 2 2

File: entity_files/building_tall.urdf (robot description, URDF)
Before this commit: robot building_tall, 1 links, 0 joints
Links:
- link building: geometry collision box size=1 1 5; visual box size=1 1 5
