Commit message: [DCL-13] PID controller now flies drone but with slight drift

File: entity_files/drone_simple.urdf (robot description, URDF)
Before this commit: robot drone_simple, 5 links, 4 joints
Links:
- link chasis: geometry collision cylinder length=0.15 radius=0.4; visual box size=0.05 0.3 0.05

Commit message: [DCL-18] Implement Lidar Sensor

File: entity_files/drone_simple.urdf (robot description, URDF)
Before this commit: robot drone_simple, 5 links, 4 joints
Links:
- removed link chasis
- added link chassis, mass 0.027; collision cylinder length=0.15 radius=0.4; visual box size=0.05 0.3 0.05
Joints:
- removed joint bl_rotor_to_chasis
- removed joint br_rotor_to_chasis
- removed joint fl_rotor_to_chasis
- removed joint fr_rotor_to_chasis
- added joint bl_rotor_to_chassis: type fixed, parent chassis, child bl_rotor
- added joint br_rotor_to_chassis: type fixed, parent chassis, child br_rotor
- added joint fl_rotor_to_chassis: type fixed, parent chassis, child fl_rotor
- added joint fr_rotor_to_chassis: type fixed, parent chassis, child fr_rotor

Commit message: [DCL-82] Basic diffusion path planning

File: entity_files/drone_simple.urdf (robot description, URDF)
Before this commit: robot drone_simple, 5 links, 4 joints
Links:
- link chassis: geometry collision cylinder length=0.15 radius=0.4; visual box size=0.03 0.03 0.2

File: entity_files/empty.urdf (robot description, URDF)
Before this commit: robot 20m_floor_t, 1 links, 0 joints
Links:
- removed link 20m_floor_obj
- added link empty_obj, mass .0; visual box size=1 1 1
