Commit message: [DCL-104] 3D cell path planning simulation created

File: entity_files/simple/1m_cube.urdf (robot description, URDF)
Before this commit: robot building_tall, 1 links, 0 joints
Links:
- removed link building
- added link cube_obj, mass 1; collision box size=0.1 0.1 0.1; visual box size=0.1 0.1 0.1

File: entity_files/simple/1m_cube_static.urdf (robot description, URDF)
Before this commit: robot building_short, 1 links, 0 joints
Links:
- removed link building
- added link cube_obj, mass 0; collision box size=1 1 1; visual box size=1 1 1
